File: Heatplate_v1.2/heatPlate.kicad_sch (KiCad schematic)
At the start: 47 parts, among them J1 Conn_01x02, J2 USB_B_Micro, Q1 SS8050, Q2 IRLR8726TRPBF, SW1 SW_Push, SW2 SW_Push, U1 NCP1117-3.3_SOT223, U2 W25Q128JVS, U3 RP2040, Y1 ABM8-272-T3

Commit message: Add files via upload
Parts:
- removed J2: USB_B_Micro, RP2040_minimal:USB_Micro-B_Amphenol_10103594-0001LF_Horizontal_modified, symbol Connector:USB_B_Micro
- added C18: 1000u, symbol Device:C
- added C19, C20, C21, C22: 680u/16V, Capacitor_THT:CP_Radial_D8.0mm_P3.50mm, symbol Device:C_Polarized_Small
- added J3: USB_C_Receptacle, Connector_USB:USB_C_Receptacle_GCT_USB4115-03-C, symbol Connector:USB_C_Receptacle
- added R13, R14, R15: 4k7, symbol Device:R
- added U4: FUSB302TMPX, WQFN14_2P5X2P5_ONS, symbol FUSB302TMPX:FUSB302TMPX
Connections:
- net VCC is gone; now on net VBUS: D1.1 (K), NT1.1, R12.2
- net +3V3: now also R13.2, R14.2, R15.2, U4.3 (VDD), U4.4 (VDD)
- net GND: now also C18.2, C19.2, C20.2, C21.2, C22.2, J3.A1 (GND), J3.A12 (GND), J3.B1 (GND), J3.B12 (GND), J3.S1 (SHIELD), U4.8 (GND), U4.9 (GND)
- net GPIO16: now also R15.1, U4.5 (INT_N)
- net GPIO17: now also R13.1, U4.6 (SCL)
- net GPIO18: now also R14.1, U4.7 (SDA)
- net VBUS: now also C18.1, C19.1, C20.1, C21.1, C22.1, J3.A4 (VBUS), J3.A9 (VBUS), J3.B4 (VBUS), J3.B9 (VBUS), U4.2 (VBUS)
- net USB_D+ renamed D+
- net D+: now also J3.A6 (D+), J3.B6 (D+)
- net USB_D- renamed D-
- net D-: now also J3.A7 (D-), J3.B7 (D-)
- new net cc1: J3.A5 (CC1), U4.10 (CC1), U4.11 (CC1)
- new net cc2: J3.B5 (CC2), U4.1 (CC2), U4.14 (CC2)
- no-connect marks 1 -> 33
Other:
- note added: "Microcontroller"
- moved on the sheet: C1, C10, C11, C12, C13, C14, C15, C16, C17, C2, C3, C4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

Commit message: Add files via upload
Parts:
- removed NT1, NT2: NetTie_2, NetTie:NetTie-2_SMD_Pad1.3mm, symbol Device:NetTie_2
- added NT3, NT4: NetTie_2, NetTie:NetTie-2_SMD_Pad0.5mm, symbol Device:NetTie_2
- C18: footprint (none) -> Capacitor_SMD:C_0402_1005Metric
- OLED1: footprint User:0.91Inch-OLED-Module -> oled:128x64OLED
- R13, R14, R15: footprint (none) -> Resistor_SMD:R_0805_2012Metric
- TEMP1: footprint Connector_PinHeader_2.54mm:PinHeader_1x03_P2.54mm_Vertical -> Package_TO_SOT_THT:TO-92_Inline
- U3: footprint RP2040_minimal:RP2040-QFN-56 -> BLUENRG-232:RP2040-QFN-56
- U4: footprint WQFN14_2P5X2P5_ONS -> Fusb3202T:WQFN14_2P5X2P5_ONS
Connections:
- net HEATPLATE: now also NT3.2, NT4.2
- net VBUS: now also NT4.1
- net at D1.2 (A), Q2.2 (D): now also NT3.1
Changed lines of the file:
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@@
 	)
 	(symbol
-		(lib_id "Device:NetTie_2")
-		(at 86.36 227.33 0)
-		(unit 1)
-		(exclude_from_sim no)
-		(in_bom no)
-		(on_board yes)
-		(dnp no)
-		(fields_autoplaced yes)
-		(property "Reference" "NT1"
-			(at 86.36 222.25 0)
-			(effects
-				(font
-					(size 1.27 1.27)
-				)
-			)
-		)
-		(property "Value" "NetTie_2"
-			(at 86.36 224.79 0)
-			(effects
-				(font
-					(size 1.27 1.27)
-				)
-			)
-		)
-		(property "Footprint" "NetTie:NetTie-2_SMD_Pad1.3mm"
-			(at 86.36 227.33 0)
-			(effects
-				(font
-					(size 1.27 1.27)
-				)
-				(hide yes)
-			)
-		)
-		(property "Datasheet" "~"
-			(at 86.36 227.33 0)
-			(effects
-				(font
-					(size 1.27 1.27)
-				)
-				(hide yes)
-			)
-		)
-		(property "Description" ""
-			(at 86.36 227.33 0)
-			(effects
-				(font
-					(size 1.27 1.27)
-				)
-				(hide yes)
-			)
-		)
-		(pin "1"
-		)
-		(pin "2"
-		)
-		(instances
-			(project "heatPlate"
-				(path "/c5775a42-ad58-4e41-8e3a-592694905d7a"
-					(reference "NT1")
-					(unit 1)
-				)
-			)
-		)
-	)
-	(symbol
 		(lib_id "power:GND")
 		(at 30.48 389.89 0)
@@
 			)
 		)
-		(property "Footprint" "Connector_PinHeader_2.54mm:PinHeader_1x03_P2.54mm_Vertical"
+		(property "Footprint" "Package_TO_SOT_THT:TO-92_Inline"
 			(at 382.27 280.67 0)
 			(effects
@@
 			)
 		)
-		(property "Footprint" ""
+		(property "Footprint" "Resistor_SMD:R_0805_2012Metric"
 			(at 408.94 144.018 90)
 			(effects
@@
 			)
 		)
-		(property "Footprint" ""
+		(property "Footprint" "Resistor_SMD:R_0805_2012Metric"
 			(at 408.94 140.208 90)
 			(effects
@@
 			)
 		)
-		(property "Footprint" ""
+		(property "Footprint" "Capacitor_SMD:C_0402_1005Metric"
 			(at 119.0752 71.12 0)
 			(effects
@@
 	)
 	(symbol
+		(lib_name "NetTie_2_1")
+		(lib_id "Device:NetTie_2")
+		(at 86.36 237.49 0)
+		(unit 1)
+		(exclude_from_sim no)
+		(in_bom no)
+		(on_board yes)
+		(dnp no)
+		(fields_autoplaced yes)
+		(property "Reference" "NT3"
+			(at 86.36 232.41 0)
+			(effects
+				(font
+					(size 1.27 1.27)
+				)
+			)
+		)
+		(property "Value" "NetTie_2"
+			(at 86.36 234.95 0)
+			(effects
+				(font
+					(size 1.27 1.27)
+				)
+			)
+		)
+		(property "Footprint" "NetTie:NetTie-2_SMD_Pad0.5mm"
+			(at 86.36 237.49 0)
+			(effects
+				(font
+					(size 1.27 1.27)
+				)
+				(hide yes)
+			)
+		)
+		(property "Datasheet" "~"
+			(at 86.36 237.49 0)
+			(effects
+				(font
+					(size 1.27 1.27)
+				)
+				(hide yes)
+			)
+		)
+		(property "Description" "Net tie, 2 pins"
+			(at 86.36 237.49 0)
+			(effects
+				(font
+					(size 1.27 1.27)
+				)
+				(hide yes)
+			)
+		)
+		(pin "2"
+		)
+		(pin "1"
+		)
+		(instances
+			(project ""
+				(path "/c5775a42-ad58-4e41-8e3a-592694905d7a"
+					(reference "NT3")
+					(unit 1)
+				)
+			)
+		)
+	)
+	(symbol
 		(lib_id "power:GND")
 		(at 309.88 322.58 0)
@@
 			)
 		)
-		(property "Footprint" "User:0.91Inch-OLED-Module"
+		(property "Footprint" "oled:128x64OLED"
 			(at 313.69 273.05 0)
 			(effects
@@
 					(size 1.27 1.27)
 				)
-				(hide yes)
 			)
 		)
@@
 			)
 		)
-		(property "Footprint" "RP2040_minimal:RP2040-QFN-56"
+		(property "Footprint" "BLUENRG-232:RP2040-QFN-56"
 			(at 332.74 132.08 0)
 			(effects
@@
 	)
 	(symbol
-		(lib_id "Device:NetTie_2")
-		(at 86.36 237.49 0)
-		(unit 1)
-		(exclude_from_sim no)
-		(in_bom no)
-		(on_board yes)
-		(dnp no)
-		(fields_autoplaced yes)
-		(property "Reference" "NT2"
-			(at 86.36 232.41 0)
-			(effects
-				(font
-					(size 1.27 1.27)
-				)
-			)
-		)
-		(property "Value" "NetTie_2"
-			(at 86.36 234.95 0)
-			(effects
-				(font
-					(size 1.27 1.27)
-				)
-			)
-		)
-		(property "Footprint" "NetTie:NetTie-2_SMD_Pad1.3mm"
-			(at 86.36 237.49 0)
-			(effects
-				(font
-					(size 1.27 1.27)
-				)
-				(hide yes)
-			)
-		)
-		(property "Datasheet" "~"
-			(at 86.36 237.49 0)
-			(effects
-				(font
-					(size 1.27 1.27)
-				)
-				(hide yes)
-			)
-		)
-		(property "Description" ""
-			(at 86.36 237.49 0)
-			(effects
-				(font
-					(size 1.27 1.27)
-				)
-				(hide yes)
-			)
-		)
-		(pin "1"
-		)
-		(pin "2"
-		)
-		(instances
-			(project "heatPlate"
-				(path "/c5775a42-ad58-4e41-8e3a-592694905d7a"
-					(reference "NT2")
-					(unit 1)
-				)
-			)
-		)
-	)
-	(symbol
 		(lib_id "Device:C_Polarized_Small")
 		(at 105.41 38.1 180)
@@
 			)
 		)
-		(property "Footprint" ""
+		(property "Footprint" "Resistor_SMD:R_0805_2012Metric"
 			(at 408.94 146.558 90)
 			(effects
@@
 	)
 	(symbol
+		(lib_name "NetTie_2_2")
+		(lib_id "Device:NetTie_2")
+		(at 86.36 227.33 0)
+		(unit 1)
+		(exclude_from_sim no)
+		(in_bom no)
+		(on_board yes)
+		(dnp no)
+		(fields_autoplaced yes)
+		(property "Reference" "NT4"
+			(at 86.36 222.25 0)
+			(effects
+				(font
+					(size 1.27 1.27)
+				)
+			)
+		)
+		(property "Value" "NetTie_2"
+			(at 86.36 224.79 0)
+			(effects
+				(font
+					(size 1.27 1.27)
+				)
+			)
+		)
+		(property "Footprint" "NetTie:NetTie-2_SMD_Pad0.5mm"
+			(at 86.36 227.33 0)
+			(effects
+				(font
+					(size 1.27 1.27)
+				)
+				(hide yes)
+			)
+		)
+		(property "Datasheet" "~"
+			(at 86.36 227.33 0)
+			(effects
+				(font
+					(size 1.27 1.27)
+				)
+				(hide yes)
+			)
+		)
+		(property "Description" "Net tie, 2 pins"
+			(at 86.36 227.33 0)
+			(effects
+				(font
+					(size 1.27 1.27)
+				)
+				(hide yes)
+			)
+		)
+		(pin "2"
+		)
+		(pin "1"
+		)
+		(instances
+			(project ""
+				(path "/c5775a42-ad58-4e41-8e3a-592694905d7a"
+					(reference "NT4")
+					(unit 1)
+				)
+			)
+		)
+	)
+	(symbol
 		(lib_id "power:+3.3V")
 		(at 297.18 271.78 0)
@@
 			)
 		)
-		(property "Footprint" "WQFN14_2P5X2P5_ONS"
+		(property "Footprint" "Fusb3202T:WQFN14_2P5X2P5_ONS"
 			(at 140.97 60.96 0)
 			(effects

Commit message: Add files via upload
Parts:
- removed J3: USB_C_Receptacle, Connector_USB:USB_C_Receptacle_GCT_USB4115-03-C, symbol Connector:USB_C_Receptacle
- added H1, H2, H5, H6: MountingHole, MountingHole:MountingHole_2.2mm_M2, symbol Mechanical:MountingHole
- added J2: USB4085-GF-A_REVB, USB_C:GCT_USB4085-GF-A_REVB, symbol USB4085-GF-A_REVB:USB4085-GF-A_REVB
Connections:
- net GND: now also J2.A1 (GND), J2.A12 (GND), J2.B1 (GND), J2.B12 (GND), J2.S1 (SHELL), J2.S2 (SHELL), J2.S3 (SHELL), J2.S4 (SHELL)
- net VBUS: now also J2.A4 (VBUS), J2.A9 (VBUS), J2.B4 (VBUS), J2.B9 (VBUS)
- net cc1: now also J2.A5 (CC1)
- net cc2: now also J2.B5 (CC2)
- new net: J2.A6 (DP1), J2.B6 (DP2)
- new net: J2.A7 (DN1), J2.B7 (DN2)
- no-connect marks 33 -> 25
Other:
- note added: "Mounting Holes"

Commit message: Add files via upload
Parts:
- removed J2: USB4085-GF-A_REVB, USB_C:GCT_USB4085-GF-A_REVB, symbol USB4085-GF-A_REVB:USB4085-GF-A_REVB
- added J3: TYPE-C-31-M-12, USB_C:HRO_TYPE-C-31-M-12, symbol TYPE-C-31-M-12:TYPE-C-31-M-12
Connections:
- net D+: now also J3.A6 (DP1), J3.B6 (DP2)
- net D-: now also J3.A7 (DN1), J3.B7 (DN2)
- net GND: now also J3.A1_B12 (GND), J3.B1_A12 (GND), J3.S1 (SHIELD), J3.S2 (SHIELD), J3.S3 (SHIELD), J3.S4 (SHIELD)
- net VBUS: now also J3.A4_B9 (VBUS), J3.B4_A9 (VBUS)
- net cc1: now also J3.A5 (CC1)
- net cc2: now also J3.B5 (CC2)

Commit message: Add files via upload
Parts:
- added C23: 100nF, Capacitor_SMD:C_0805_2012Metric, symbol Device:C_Small
- added F1: 5A, Fuse:Fuse_2920_7451Metric, symbol Device:Polyfuse_Small
Connections:
- net GND: now also C23.2; no longer R9.1, SW2.1, U3.9 (GPIO7)
- net VBUS: now also F1.2; no longer J3.A4_B9 (VBUS), J3.B4_A9 (VBUS)
- new net: F1.1, J3.A4_B9 (VBUS), J3.B4_A9 (VBUS)
- new net GPIO7: C23.1, R9.1, SW2.1, U3.9 (GPIO7)
Other:
- moved on the sheet: C20, C21

Commit message: Minor placement changes
Connections:
- net +VDC: now reaches F1.1, J3.A4_B9 (VBUS), J3.B4_A9 (VBUS)
Changed lines of the file:
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@@
 	)
 	(junction
+		(at 58.42 40.64)
+		(diameter 0)
+		(color 0 0 0 0)
+	)
+	(junction
 		(at 358.14 68.58)
 		(diameter 0)
@@
 	)
 	(junction
-		(at 109.22 48.26)
-		(diameter 0)
-		(color 0 0 0 0)
-	)
-	(junction
 		(at 67.31 245.11)
 		(diameter 0)
@@
 	(wire
 		(pts
-			(xy 109.22 40.64) (xy 109.22 48.26)
+			(xy 109.22 40.64) (xy 109.22 63.5)
 		)
 		(stroke
@@
 	(wire
 		(pts
+			(xy 118.11 63.5) (xy 140.97 63.5)
+		)
+		(stroke
+			(width 0)
+			(type default)
+		)
+	)
+	(wire
+		(pts
 			(xy 411.48 48.26) (xy 422.91 48.26)
 		)
@@
 	(wire
 		(pts
+			(xy 58.42 38.1) (xy 58.42 40.64)
+		)
+		(stroke
+			(width 0)
+			(type default)
+		)
+	)
+	(wire
+		(pts
 			(xy 388.62 59.69) (xy 377.19 59.69)
 		)
@@
 	(wire
 		(pts
-			(xy 109.22 48.26) (xy 109.22 63.5)
-		)
-		(stroke
-			(width 0)
-			(type default)
-		)
-	)
-	(wire
-		(pts
 			(xy 383.54 142.24) (xy 405.13 142.24)
 		)
@@
 		)
 	)
-	(polyline
+	(wire
 		(pts
-			(xy 227.33 243.84) (xy 227.33 382.27)
+			(xy 118.11 59.69) (xy 118.11 63.5)
 		)
 		(stroke
@@
 		)
 	)
-	(wire
+	(polyline
 		(pts
-			(xy 118.11 63.5) (xy 140.97 63.5)
+			(xy 227.33 243.84) (xy 227.33 382.27)
 		)
 		(stroke
@@
 	)
 	(symbol
+		(lib_id "power:+VDC")
+		(at 58.42 38.1 0)
+		(unit 1)
+		(exclude_from_sim no)
+		(in_bom yes)
+		(on_board yes)
+		(dnp no)
+		(fields_autoplaced yes)
+		(property "Reference" "#PWR051"
+			(at 58.42 40.64 0)
+			(effects
+				(font
+					(size 1.27 1.27)
+				)
+				(hide yes)
+			)
+		)
+		(property "Value" "+VDC"
+			(at 58.42 30.48 0)
+			(effects
+				(font
+					(size 1.27 1.27)
+				)
+			)
+		)
+		(property "Footprint" ""
+			(at 58.42 38.1 0)
+			(effects
+				(font
+					(size 1.27 1.27)
+				)
+				(hide yes)
+			)
+		)
+		(property "Datasheet" ""
+			(at 58.42 38.1 0)
+			(effects
+				(font
+					(size 1.27 1.27)
+				)
+				(hide yes)
+			)
+		)
+		(property "Description" "Power symbol creates a global label with name \"+VDC\""
+			(at 58.42 38.1 0)
+			(effects
+				(font
+					(size 1.27 1.27)
+				)
+				(hide yes)
+			)
+		)
+		(pin "1"
+		)
+		(instances
+			(project ""
+				(path "/c5775a42-ad58-4e41-8e3a-592694905d7a"
+					(reference "#PWR051")
+					(unit 1)
+				)
+			)
+		)
+	)
+	(symbol
 		(lib_id "Device:C")
 		(at 322.58 53.34 0)
@@
 		(lib_name "VBUS_1")
 		(lib_id "power:VBUS")
-		(at 109.22 48.26 270)
+		(at 118.11 59.69 0)
 		(unit 1)
 		(exclude_from_sim no)
@@
 		(on_board yes)
 		(dnp no)
-		(fields_autoplaced yes)
 		(property "Reference" "#PWR045"
-			(at 105.41 48.26 0)
+			(at 118.11 63.5 0)
 			(effects
 				(font
@@
 		)
 		(property "Value" "VBUS"
-			(at 113.03 48.2599 90)
+			(at 110.49 58.928 0)
 			(effects
 				(font
@@
 		)
 		(property "Footprint" ""
-			(at 109.22 48.26 0)
+			(at 118.11 59.69 0)
 			(effects
 				(font
@@
 		)
 		(property "Datasheet" ""
-			(at 109.22 48.26 0)
+			(at 118.11 59.69 0)
 			(effects
 				(font
@@
 		)
 		(property "Description" "Power symbol creates a global label with name \"VBUS\""
-			(at 109.22 48.26 0)
+			(at 118.11 59.69 0)
 			(effects
 				(font

Commit message: components change to 0402
compo
Parts:
- C17, C3, C4: footprint Capacitor_SMD:C_0805_2012Metric -> Capacitor_SMD:C_0402_1005Metric
- R10, R11, R12, R13, R14, R15, R6, R7, R8, R9: footprint Resistor_SMD:R_0805_2012Metric -> Resistor_SMD:R_0402_1005Metric
Changed lines of the file:
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@@
 			)
 		)
-		(property "Footprint" "Capacitor_SMD:C_0805_2012Metric"
+		(property "Footprint" "Capacitor_SMD:C_0402_1005Metric"
 			(at 110.1852 137.16 0)
 			(effects
@@
 			)
 		)
-		(property "Footprint" "Capacitor_SMD:C_0805_2012Metric"
+		(property "Footprint" "Capacitor_SMD:C_0402_1005Metric"
 			(at 80.9752 138.43 0)
 			(effects
@@
 			)
 		)
-		(property "Footprint" "Resistor_SMD:R_0805_2012Metric"
+		(property "Footprint" "Resistor_SMD:R_0402_1005Metric"
 			(at 408.94 144.018 90)
 			(effects
@@
 			)
 		)
-		(property "Footprint" "Resistor_SMD:R_0805_2012Metric"
+		(property "Footprint" "Resistor_SMD:R_0402_1005Metric"
 			(at 408.94 140.208 90)
 			(effects
@@
 			)
 		)
-		(property "Footprint" "Resistor_SMD:R_0805_2012Metric"
+		(property "Footprint" "Resistor_SMD:R_0402_1005Metric"
 			(at 264.16 318.77 0)
 			(effects
@@
 			)
 		)
-		(property "Footprint" "Resistor_SMD:R_0805_2012Metric"
+		(property "Footprint" "Resistor_SMD:R_0402_1005Metric"
 			(at 309.88 307.34 0)
 			(effects
@@
 			)
 		)
-		(property "Footprint" "Resistor_SMD:R_0805_2012Metric"
+		(property "Footprint" "Resistor_SMD:R_0402_1005Metric"
 			(at 264.16 302.26 0)
 			(effects
@@
 			)
 		)
-		(property "Footprint" "Resistor_SMD:R_0805_2012Metric"
+		(property "Footprint" "Resistor_SMD:R_0402_1005Metric"
 			(at 52.07 252.73 0)
 			(effects
@@
 			)
 		)
-		(property "Footprint" "Resistor_SMD:R_0805_2012Metric"
+		(property "Footprint" "Resistor_SMD:R_0402_1005Metric"
 			(at 67.31 240.03 0)
 			(effects
@@
 			)
 		)
-		(property "Footprint" "Resistor_SMD:R_0805_2012Metric"
+		(property "Footprint" "Resistor_SMD:R_0402_1005Metric"
 			(at 408.94 146.558 90)
 			(effects
@@
 			)
 		)
-		(property "Footprint" "Resistor_SMD:R_0805_2012Metric"
+		(property "Footprint" "Resistor_SMD:R_0402_1005Metric"
 			(at 309.88 340.36 0)
 			(effects
@@
 			)
 		)
-		(property "Footprint" "Capacitor_SMD:C_0805_2012Metric"
+		(property "Footprint" "Capacitor_SMD:C_0402_1005Metric"
 			(at 309.88 317.5 0)
 			(effects
@@
 			)
 		)
-		(property "Footprint" "Resistor_SMD:R_0805_2012Metric"
+		(property "Footprint" "Resistor_SMD:R_0402_1005Metric"
 			(at 57.15 247.65 0)
 			(effects

Commit message: components change to 0402
Parts:
- C23: footprint Capacitor_SMD:C_0805_2012Metric -> Capacitor_SMD:C_0402_1005Metric
Changed lines of the file:
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@@
 			)
 		)
-		(property "Footprint" "Capacitor_SMD:C_0805_2012Metric"
+		(property "Footprint" "Capacitor_SMD:C_0402_1005Metric"
 			(at 309.88 350.52 0)
 			(effects
