File: Heatplate_v1.2/heatPlate.kicad_sch (KiCad schematic)
At the start: 66 parts, among them J1 Conn_01x02, J2 SM03B-SRSS-TB, J3 TYPE-C-31-M-12, Q1 SS8050, Q2 IRLR8726TRPBF, SW1 SW_Push, SW2 SW_Push, SW3 SW_Push, U1 NCP1117-3.3_SOT223, U2 W25Q128JVS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

Commit message: sd-card added
Parts:
- added J4: MSD-1-A, MSD-1-A:CUI_MSD-1-A, symbol MSD-1-A:MSD-1-A
Connections:
- net +3V3: now also J4.4 (VDD)
- net GND: now also J4.6 (VSS), J4.G1 (COVER_GND), J4.G2 (COVER_GND), J4.G3 (COVER_GND), J4.G4 (COVER_GND)
- net GPIO0: now also J4.2 (CD/DAT3)
- net GPIO1: now also J4.3 (CMD)
- net GPIO10: now also J4.CD
- net GPIO2: now also J4.7 (DAT0)
- net GPIO22: now also R2.2
- net GPIO23: now also R17.2
- net GPIO3: now also J4.5 (CLK)
- no-connect marks 21 -> 16
Other:
- note added: "SD-Card"

Commit message: sd_card
Parts:
- J4: footprint MSD-1-A:CUI_MSD-1-A -> sd_card:microSD_External_Pin
Changed lines of the file:
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@@
 			)
 		)
-		(property "Footprint" "MSD-1-A:CUI_MSD-1-A"
+		(property "Footprint" "sd_card:microSD_External_Pin"
 			(at 135.89 250.19 0)
 			(effects
