File: Heatplate_v1.2/heatPlate.kicad_pcb (KiCad board)
At the start: 2 copper layers, 112 x 176 mm, 67 parts, among them J1 Conn_01x02, J2 SM03B-SRSS-TB, J3 TYPE-C-31-M-12, J4 MSD-1-A, Q1 SS8050, Q2 IRLR8726TRPBF, SW1 SW_Push, SW2 SW_Push, SW3 SW_Push, U1 NCP1117-3.3_SOT223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

Commit message: minor changes
Parts:
- moved C17 153.5 mm to (294.1, 69.5)
- moved C10 153.5 mm to (285.9, 67.2)
- moved C11 153.5 mm to (273.5, 66.6)
- moved C12 153.5 mm to (288.0, 62.7)
- moved C13 153.5 mm to (248.8, 62.5)
- moved C14 153.5 mm to (248.8, 60.5)
- moved C15 153.5 mm to (286.2, 62.8)
- moved C16 153.5 mm to (273.0, 70.2)
- moved C23 153.5 mm to (287.9, 68.8)
- moved C6 153.5 mm to (279.1, 59.5)
- moved C7 153.5 mm to (284.5, 62.8)
- moved C8 153.5 mm to (285.9, 65.2)
- moved C9 153.5 mm to (282.8, 62.7)
- moved LED1 153.5 mm to (289.5, 76.5)
- moved R14 153.5 mm to (286.5, 72.0)
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Other:
- board size 112 x 176 mm -> 112 x 185.4 mm

Commit message: minor changes
Parts:
- added C24: 10u, Capacitor_SMD:C_0603_1608Metric, F.Cu at (150.9, 68.2)
- added R18: ~, Resistor_SMD:R_0603_1608Metric, F.Cu at (150.9, 70.2)
- moved R6 179.0 mm to (113.2, 66.8), turned to 180 degrees
- moved R7 174.8 mm to (113.2, 68.5)
- moved C23 174.7 mm to (113.2, 65.0), turned to 180 degrees
- moved R4 174.3 mm to (106.5, 59.5), turned to 90 degrees
- moved R5 168.5 mm to (113.9, 62.2), turned to 0 degrees
- moved C10 161.7 mm to (124.5, 58.0), turned to 90 degrees
- moved C12 160.1 mm to (128.0, 58.0)
- moved C15 160.1 mm to (126.2, 58.0)
- moved C9 160.1 mm to (122.8, 58.0)
- moved R14 156.9 mm to (129.6, 68.6)
- moved C8 156.8 mm to (129.2, 61.2)
- moved C11 156.2 mm to (117.5, 58.0), turned to 90 degrees
- moved C17 154.7 mm to (140.0, 55.8), turned to 180 degrees
- moved R9 152.2 mm to (136.4, 55.8)
- moved C7 152.0 mm to (132.5, 61.0)
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Connections:
- J4 pad 2: /GPIO0 -> /GPIO3
- J4 pad 3: /GPIO1 -> /GPIO13
- J4 pad 5: /GPIO3 -> /GPIO14
- J4 pad 7: /GPIO2 -> /GPIO0

Commit message: minor changes
Parts:
- moved F1 0.65 mm to (65.2, 69.4)
Changed lines of the file:
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@@
 	(footprint "Fuse:Fuse_2920_7451Metric"
 		(layer "F.Cu")
-		(at 65.25 68.75 90)
+		(at 65.2 69.4 90)
 		(descr "Fuse SMD 2920 (7451 Metric), square (rectangular) end terminal, IPC_7351 nominal, (Body size from: http://www.megastar.com/products/fusetronic/polyswitch/PDF/smd2920.pdf), generated with kicad-footprint-generator")
 		(tags "fuse")

Commit message: routing
Parts:
- moved J2 35.5 mm to (108.4, 49.6), turned to 180 degrees
- moved R3 14.6 mm to (123.6, 71.8)
- moved R1 9.36 mm to (115.4, 53.2), turned to 0 degrees
- moved LED1 5.98 mm to (140.3, 61.4)
- moved R5 4.74 mm to (109.6, 64.2)
- moved R4 4.38 mm to (109.6, 62.6), turned to 0 degrees
- moved U2 4.33 mm to (108.6, 56.6)
- moved J1 3.18 mm to (116.4, 48.8), turned to 90 degrees
- moved C2 2.57 mm to (139.8, 70.4)
- moved C5 2.23 mm to (123.4, 52.8)
- moved SW2 1.80 mm to (134.7, 53.0)
- moved SW1 1.45 mm to (145.1, 53.0)
- moved C16 0.99 mm to (129.6, 57.0)
- moved C10 0.98 mm to (124.4, 57.0)
- moved C12 0.98 mm to (127.9, 57.0)
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Routing:
- net /GPIO14: track 0.00 -> 51.9 mm, vias 0 -> 3
- net /GPIO13: track 0.00 -> 49.5 mm, vias 0 -> 2
- net /GPIO6: track 0.00 -> 48.3 mm, vias 0 -> 2
- net /GPIO3: track 0.00 -> 46.8 mm, vias 0 -> 2
- net /GPIO21: track 0.00 -> 38.5 mm
- net /GPIO7: track 0.00 -> 36.2 mm, vias 0 -> 2
- net /QSPI_SS: track 0.00 -> 35.8 mm
- net /GPIO20: track 0.00 -> 35.1 mm
- net +3V3: track 0.00 -> 26.3 mm
- net /QSPI_SD1: track 0.00 -> 24.7 mm
- net /QSPI_SD2: track 0.00 -> 23.4 mm
- net GND: track 0.00 -> 14.2 mm
- net /QSPI_SD3: track 0.00 -> 14.0 mm
- net /QSPI_SCLK: track 0.00 -> 13.0 mm
- net /QSPI_SD0: track 0.00 -> 11.6 mm
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- added copper zone on B.Cu, net GND
- added copper zone on F.Cu, net VBUS

Commit message: routing
Parts:
- moved R10 3.63 mm to (97.0, 59.4)
- moved R4 1.80 mm to (109.6, 64.4)
- moved R5 1.60 mm to (109.6, 62.6)
- moved R11 1.22 mm to (95.2, 57.2)
- moved C4 1.15 mm to (91.6, 57.4)
- turned F1 to -90 degrees
Routing:
- net /GPIO16: track 5.49 -> 64.3 mm, vias 0 -> 2
- net /GPIO17: track 4.05 -> 62.1 mm, vias 0 -> 2
- net /GPIO18: track 2.82 -> 59.5 mm, vias 0 -> 2
- net /D-: track 0.00 -> 47.0 mm
- net /D+: track 0.00 -> 46.2 mm
- net /SWCLK: track 0.00 -> 41.1 mm, vias 0 -> 2
- net VBUS: track 1.96 -> 37.7 mm, vias 0 -> 1
- net Net-(Q1-C): track 0.00 -> 21.8 mm
- net +VDC: track 0.00 -> 16.9 mm
- net Net-(U3-USB_DM): track 0.00 -> 16.1 mm, vias 0 -> 2
- net Net-(U3-USB_DP): track 0.00 -> 15.1 mm, vias 0 -> 2
- net /cc1: track 0.00 -> 12.7 mm, vias 0 -> 2
- net /cc2: track 0.00 -> 11.2 mm
- net GND: track 14.2 -> 16.9 mm
- net /SWD: track 0.00 -> 1.30 mm, vias 0 -> 1
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- added copper zone on F.Cu, net HEATPLATE

Commit message: routing
Parts:
- moved C5 8.79 mm to (129.2, 59.4), turned to 0 degrees
- moved LED1 4.64 mm to (144.8, 60.2)
- moved C7 2.00 mm to (132.6, 63.0), turned to 0 degrees
- moved R4 2.00 mm to (109.6, 66.4)
- moved R5 1.40 mm to (108.6, 63.6)
- moved R17 0.80 mm to (102.2, 51.8), turned to -90 degrees
- turned R16 to 180 degrees
Routing:
- net /GPIO23: track 0.00 -> 64.5 mm, vias 0 -> 2
- net /RUN: track 0.00 -> 51.5 mm, vias 0 -> 2
- net /QSPI_SS: track 35.8 -> 78.4 mm, vias 0 -> 2
- net Net-(LED1B-A2): track 0.00 -> 42.5 mm, vias 0 -> 2
- net Net-(LED1A-A1): track 0.00 -> 40.6 mm, vias 0 -> 4
- net /SWD: track 1.30 -> 41.1 mm, vias 1 -> 2
- net VBUS: track 37.7 -> 74.0 mm
- net GND: track 16.9 -> 50.0 mm
- net Net-(C2-Pad1): track 0.00 -> 26.4 mm
- net Net-(D1-A): track 1.96 -> 17.2 mm
- net +1V1: track 0.00 -> 14.2 mm, vias 0 -> 2
- net Net-(R16-Pad2): track 0.00 -> 9.41 mm
- net /GPIO9: track 0.00 -> 5.48 mm
- net /GPIO8: track 0.00 -> 5.28 mm
- net Net-(U3-USB_DP): track 15.1 -> 17.1 mm
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
Commit message: routing
Parts:
- moved R3 0.40 mm to (123.6, 72.2)
- moved C1 0.28 mm to (122.0, 71.6)
Routing:
- net /GPIO26_ADC0: track 0.00 -> 64.3 mm, vias 0 -> 3
- net /GPIO4: track 0.00 -> 58.4 mm, vias 0 -> 4
- net /GPIO5: track 0.00 -> 43.8 mm, vias 0 -> 3
- net /GPIO15: track 0.00 -> 27.8 mm, vias 0 -> 4
- net Net-(Q1-B): track 0.00 -> 15.9 mm, vias 0 -> 2
- net GND: track 50.0 -> 64.0 mm, vias 0 -> 2

Commit message: routing
Parts:
- moved C24 33.7 mm to (123.4, 48.8)
- moved TEMP3 0.30 mm to (169.9, 73.5)
Routing:
- net /GPIO0: track 0.00 -> 69.9 mm, vias 0 -> 2
- net GND: track 64.0 -> 122.0 mm, vias 2 -> 8
- net +3V3: track 29.2 -> 86.5 mm, vias 0 -> 4
- net +3.3V: track 0.00 -> 51.0 mm, vias 0 -> 1
- net /GPIO4: track 58.4 -> 53.8 mm
- net /GPIO3: track 46.8 -> 45.9 mm
Other:
- outline, holes or cut-outs redrawn
